Commit message: Added Laser

File: urdf/2wr.xacro (robot description, xacro)
@@ -1,53 +1,7 @@
 <?xml version="1.0" ?>
 <robot name="2wr" xmlns:xacro="http://www.ros.org/wiki/xacro">
-  <material name="black">
-    <color rgba="0.0 0.0 0.0 1.0"/>
-  </material>
-  <material name="blue">
-    <color rgba="0.203125 0.23828125 0.28515625 1.0"/>
-  </material>
-  <material name="green">
-    <color rgba="0.0 0.8 0.0 1.0"/>
-  </material>
-  <material name="grey">
-    <color rgba="0.2 0.2 0.2 1.0"/>
-  </material>
-  <material name="orange">
-    <color rgba="1.0 0.423529411765 0.0392156862745 1.0"/>
-  </material>
-  <material name="brown">
-    <color rgba="0.870588235294 0.811764705882 0.764705882353 1.0"/>
-  </material>
-  <material name="red">
-    <color rgba="0.80078125 0.12890625 0.1328125 1.0"/>
-  </material>
-  <material name="white">
-    <color rgba="1.0 1.0 1.0 1.0"/>
-  </material>
-  <gazebo reference="link_chassis">
-    <material>Gazebo/Orange</material>
-  </gazebo>
-  <gazebo reference="link_left_wheel">
-    <material>Gazebo/Blue</material>
-  </gazebo>
-  <gazebo reference="link_right_wheel">
-    <material>Gazebo/Blue</material>
-  </gazebo>
-  <gazebo> <!-- Can do this way as it is a already done structure or http://wiki.ros.org/urdf/Tutorials/Using%20a%20URDF%20in%20Gazebo -->
-    <plugin filename="libgazebo_ros_diff_drive.so" name="differential_drive_controller">
-      <legacyMode>false</legacyMode>
-      <alwaysOn>true</alwaysOn>
-      <updateRate>20</updateRate>
-      <leftJoint>joint_left_wheel</leftJoint>
-      <rightJoint>joint_right_wheel</rightJoint>
-      <wheelSeparation>0.3</wheelSeparation>
-      <wheelDiameter>0.2</wheelDiameter>
-      <torque>0.1</torque>
-      <commandTopic>cmd_vel</commandTopic>
-      <odometryTopic>odom</odometryTopic>
-      <odometryFrame>odom</odometryFrame>
-      <robotBaseFrame>link_chassis</robotBaseFrame>
-    </plugin>
-  </gazebo>
+  <xacro:include filename="$(find two_wheeled_robot)/urdf/materials.xacro" />
+  <xacro:include filename="$(find two_wheeled_robot)/urdf/2wr.gazebo" />
+  <xacro:include filename="$(find two_wheeled_robot)/urdf/macros.xacro" />
   <link name="link_chassis">
     <!-- pose and inertial -->
@@ -95,57 +49,32 @@
     </visual>
   </link>
-  <link name="link_right_wheel">
+  <link name="sensor_laser">
     <inertial>
-      <mass value="0.2"/>
-      <origin rpy="0 1.5707 1.5707" xyz="0 0 0"/>
-      <inertia ixx="0.000526666666667" ixy="0" ixz="0" iyy="0.000526666666667" iyz="0" izz="0.001"/>
+        <origin xyz="0 0 0" rpy="0 0 0" />
+        <mass value="1" />
+        <xacro:cylinder_inertia mass="1" r="0.05" l="0.1" />
     </inertial>
-    <collision name="link_right_wheel_collision">
-      <origin rpy="0 1.5707 1.5707" xyz="0 0 0"/>
-      <geometry>
-        <cylinder length="0.04" radius="0.1"/>
-      </geometry>
+    <visual>
+        <origin xyz="0 0 0" rpy="0 0 0" />
+        <geometry>
+          <cylinder radius="0.05" length="0.1"/>
+        </geometry>
+        <material name="white" />
+    </visual>
+    <collision>
+        <origin xyz="0 0 0" rpy="0 0 0"/>
+        <geometry>
+          <cylinder radius="0.05" length="0.1"/>
+        </geometry>
     </collision>
-    <visual name="link_right_wheel_visual">
-      <origin rpy="0 1.5707 1.5707" xyz="0 0 0"/>
-      <geometry>
-        <cylinder length="0.04" radius="0.1"/>
-      </geometry>
-    </visual>
-  </link>
-  <joint name="joint_right_wheel" type="continuous">
-    <origin rpy="0 0 0" xyz="-0.05 0.15 0"/>
-    <child link="link_right_wheel"/>
+ </link>
+  <joint name="joint_sensor_laser" type="fixed">
+    <origin xyz="0.15 0 0.05" rpy="0 0 0"/>
     <parent link="link_chassis"/>
-    <axis rpy="0 0 0" xyz="0 1 0"/>
-    <limit effort="10000" velocity="1000"/>
-    <joint_properties damping="1.0" friction="1.0"/>
+    <child link="sensor_laser"/>
   </joint>
-  <link name="link_left_wheel">
-    <inertial>
-      <mass value="0.2"/>
-      <origin rpy="0 1.5707 1.5707" xyz="0 0 0"/>
-      <inertia ixx="0.000526666666667" ixy="0" ixz="0" iyy="0.000526666666667" iyz="0" izz="0.001"/>
-    </inertial>
-    <collision name="link_left_wheel_collision">
-      <origin rpy="0 1.5707 1.5707" xyz="0 0 0"/>
-      <geometry>
-        <cylinder length="0.04" radius="0.1"/>
-      </geometry>
-    </collision>
-    <visual name="link_left_wheel_visual">
-      <origin rpy="0 1.5707 1.5707" xyz="0 0 0"/>
-      <geometry>
-        <cylinder length="0.04" radius="0.1"/>
-      </geometry>
-    </visual>
-  </link>
-  <joint name="joint_left_wheel" type="continuous">
-    <origin rpy="0 0 0" xyz="-0.05 -0.15 0"/>
-    <child link="link_left_wheel"/>
-    <parent link="link_chassis"/>
-    <axis rpy="0 0 0" xyz="0 1 0"/>
-    <limit effort="10000" velocity="1000"/>
-    <joint_properties damping="1.0" friction="1.0"/>
-  </joint>
+  <xacro:link_wheel name="link_right_wheel" />
+  <xacro:joint_wheel name="joint_right_wheel" child="link_right_wheel" origin_xyz="-0.05 0.15 0" />
+  <xacro:link_wheel name="link_left_wheel" />
+  <xacro:joint_wheel name="joint_left_wheel" child="link_left_wheel" origin_xyz="-0.05 -0.15 0" />
 </robot>

Commit message: Updated working version of the code

File: urdf/2wr.xacro (robot description, xacro)
@@ -23,5 +23,5 @@
         <box size="0.5 0.3 0.07"/>
       </geometry>
-      <material name="blue"/>
+      <material name="orange"/>
     </visual>
     <!-- caster front -->
@@ -47,4 +47,5 @@
         <sphere radius="0.05"/>
       </geometry>
+      <material name="white"/>
     </visual>
   </link>
@@ -74,4 +75,166 @@
     <child link="sensor_laser"/>
   </joint>
+  <link name="camera_link">
+    <inertial>
+        <mass value="1e-5" />
+        <origin xyz="0 0 0" rpy="0 0 0"/>
+        <inertia ixx="1e-6" ixy="0" ixz="0" iyy="1e-6" iyz="0" izz="1e-6" />
+    </inertial>
+    <visual>
+        <origin xyz="0 0 0" rpy="0 0 0" />
+        <geometry>
+          <box size="0.02 0.1 0.02"/>
+        </geometry>
+        <material name="white" />
+    </visual>
+    <collision>
+        <origin xyz="0 0 0" rpy="0 0 0"/>
+        <geometry>
+          <box size="0.02 0.1 0.02"/>
+        </geometry>
+    </collision>
+ </link>
+ <joint name="joint_camera" type="fixed">
+   <origin xyz="0.25 0 0" rpy="0 0 0"/>
+   <parent link="link_chassis"/>
+   <child link="camera_link"/>
+ </joint>
+ <link name="base_link">
+  <visual>
+    <geometry>
+      <cylinder radius="0.05" length="0.1"/>
+    </geometry>
+    <material name="orange"/>
+    <origin rpy="0 0 0" xyz="0 0 -0.025"/>
+  </visual>
+</link>
+<joint name="joint_base_arm" type="fixed">
+  <origin xyz="0.15 0 0.175" rpy="0 0 -1.570796"/>
+  <parent link="link_chassis"/>
+  <child link="base_link"/>
+</joint>
+<link name="link1">
+  <visual>
+    <geometry>
+      <mesh filename="package://two_wheeled_robot/meshes/base.stl"/>
+    </geometry>
+    <material name="orange"/>
+  </visual>
+</link>
+<link name="link2">
+  <visual>
+    <geometry>
+      <mesh filename="package://two_wheeled_robot/meshes/shoulder.stl"/>
+    </geometry>
+    <material name="orange"/>
+    <origin rpy="0 0 0" xyz="0 0 -0.0505"/>
+  </visual>
+</link>
+<link name="link3">
+  <visual>
+    <geometry>
+      <mesh filename="package://two_wheeled_robot/meshes/elbow.stl"/>
+    </geometry>
+    <material name="orange"/>
+    <origin rpy="0 0 0" xyz="0 0 -0.1705"/>
+  </visual>
+</link>
+<link name="link4">
+  <visual>
+    <geometry>
+      <mesh filename="package://two_wheeled_robot/meshes/wrist_pitch.stl"/>
+    </geometry>
+    <material name="orange"/>
+    <origin rpy="0 0 0" xyz="0 0 -0.2905"/>
+  </visual>
+</link>
+<link name="link5">
+  <visual>
+    <geometry>
+      <mesh filename="package://two_wheeled_robot/meshes/wrist_roll.stl"/>
+    </geometry>
+    <material name="white"/>
+    <origin rpy="0 0 0" xyz="0 0 -0.3505"/>
+  </visual>
+</link>
+<link name="gripper_base">
+  <visual>
+    <geometry>
+      <mesh filename="package://two_wheeled_robot/meshes/gripper_base.stl"/>
+    </geometry>
+    <material name="white"/>
+    <origin rpy="0 0 0" xyz="0 0 -0.357"/>
+  </visual>
+</link>
+<link name="gripper_fix">
+  <visual>
+    <geometry>
+      <mesh filename="package://two_wheeled_robot/meshes/gripper_fix.stl"/>
+    </geometry>
+    <material name="white"/>
+    <origin rpy="0 0 0" xyz="0 0 -0.36399"/>
+  </visual>
+</link>
+<link name="gripper_movable">
+  <visual>
+    <geometry>
+      <mesh filename="package://two_wheeled_robot/meshes/gripper_movable.stl"/>
+    </geometry>
+    <material name="white"/>
+    <origin rpy="0 0 0" xyz="-0.01559 0 -0.36399"/>
+  </visual>
+</link>
+<joint name="base" type="revolute">
+  <axis xyz="0 0 -1"/>
+  <limit effort="1000.0" lower="0.0" upper="3.141592653589793" velocity="4.0"/>
+  <origin rpy="0 0 0" xyz="0 0 0"/>
+  <parent link="base_link"/>
+  <child link="link1"/>
+</joint>
+<joint name="shoulder" type="revolute">
+  <axis xyz="1 0 0"/>
+  <limit effort="1000.0" lower="0.2617993877991494" upper="2.8797932657906435" velocity="4.0"/>
+  <origin rpy="-1.5707963267948966 0 0" xyz="0 0 0.0505"/>
+  <parent link="link1"/>
+  <child link="link2"/>
+</joint>
+ <joint name="elbow" type="revolute">
+  <axis xyz="1 0 0"/>
+  <limit effort="1000.0" lower="0" upper="3.141592653589793" velocity="4.0"/>
+  <origin rpy="-1.5707963267948966 0 0" xyz="0 0 0.1205"/>
+  <parent link="link2"/>
+  <child link="link3"/>
+</joint>
+<joint name="wrist_pitch" type="revolute">
+  <axis xyz="1 0 0"/>
+  <limit effort="1000.0" lower="0" upper="3.141592653589793" velocity="4.0"/>
+  <origin rpy="-1.5707963267948966 0 0" xyz="0 0 0.1205"/>
+  <parent link="link3"/>
+  <child link="link4"/>
+</joint>
+<joint name="wrist_roll" type="revolute">
+  <axis xyz="0 0 -1"/>
+  <limit effort="1000.0" lower="0.0" upper="3.141592653589793" velocity="4.0"/>
+  <origin rpy="0 0 0" xyz="0 0.0 0.06"/>
+  <parent link="link4"/>
+  <child link="link5"/>
+</joint>
+<joint name="gripper_base" type="fixed">
+  <origin rpy="0 0 0" xyz="0 0.0 0.0065"/>
+  <parent link="link5"/>
+  <child link="gripper_base"/>
+</joint>
+<joint name="gripper_fix" type="fixed">
+  <origin rpy="0 0 0" xyz="0 0.0 0.007"/>
+  <parent link="gripper_base"/>
+  <child link="gripper_fix"/>
+</joint>
+<joint name="gripper_movable" type="revolute">
+  <axis xyz="0 -1 0"/>
+  <limit effort="1000.0" lower="0.17453292519943295" upper="1.2740903539558606" velocity="4.0"/>
+  <origin rpy="0 0 0" xyz="0.01559 0 0.007"/>
+  <parent link="gripper_base"/>
+  <child link="gripper_movable"/>
+</joint>
   <xacro:link_wheel name="link_right_wheel" />
   <xacro:joint_wheel name="joint_right_wheel" child="link_right_wheel" origin_xyz="-0.05 0.15 0" />

File: urdf/macros.xacro (robot description, xacro)
@@ -19,4 +19,5 @@
                 <cylinder length="0.04" radius="0.1"/>
               </geometry>
+              <material name="white"/>
             </visual>
         </link>

Commit message: Update

File: urdf/2wr.xacro (robot description, xacro)
@@ -103,5 +103,5 @@
   <visual>
     <geometry>
-      <cylinder radius="0.05" length="0.1"/>
+      <cylinder radius="0.05" length="0.25"/>
     </geometry>
     <material name="orange"/>
@@ -110,5 +110,5 @@
 </link>
 <joint name="joint_base_arm" type="fixed">
-  <origin xyz="0.15 0 0.175" rpy="0 0 -1.570796"/>
+  <origin xyz="0 0 0.175" rpy="0 0 -1.570796"/>
   <parent link="link_chassis"/>
   <child link="base_link"/>
@@ -238,6 +238,10 @@
 </joint>
   <xacro:link_wheel name="link_right_wheel" />
-  <xacro:joint_wheel name="joint_right_wheel" child="link_right_wheel" origin_xyz="-0.05 0.15 0" />
+  <xacro:joint_wheel name="joint_right_wheel" child="link_right_wheel" origin_xyz="-0.15 0.15 -0.10" />
   <xacro:link_wheel name="link_left_wheel" />
-  <xacro:joint_wheel name="joint_left_wheel" child="link_left_wheel" origin_xyz="-0.05 -0.15 0" />
+  <xacro:joint_wheel name="joint_left_wheel" child="link_left_wheel" origin_xyz="-0.15 -0.15 -0.10" />
+  <xacro:link_wheel name="link_right_wheel_front" />
+  <xacro:joint_wheel name="joint_right_wheel_front" child="link_right_wheel_front" origin_xyz="0.15 0.15 -0.10" />
+  <xacro:link_wheel name="link_left_wheel_front" />
+  <xacro:joint_wheel name="joint_left_wheel_front" child="link_left_wheel_front" origin_xyz="0.15 -0.15 -0.10" />
 </robot>

File: urdf/macros.xacro (robot description, xacro)
@@ -19,5 +19,5 @@
                 <cylinder length="0.04" radius="0.1"/>
               </geometry>
-              <material name="white"/>
+              <material name="black"/>
             </visual>
         </link>
